File: pwm-fan-control.kicad_pcb (KiCad board)
At the start: 2 copper layers, 17.4 x 26.9 mm, 14 parts, among them J1 12V_IN, J2 FAN_OUT, J3 Conn_ESP_PROG_1.27mm_TagConne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, J4 ADJ_IN, Q1 NMOS (100V 1.5A 2Vth), U1 NCP1117-5.0_SOT223, U2 ATtiny10-TS

Commit message: Layout done
Parts:
- moved C4 11.3 mm to (88.7, 72.5), turned to -90 degrees
- moved R1 5.75 mm to (93.6, 58.1), turned to 90 degrees
- moved Q1 1.00 mm to (90.2, 58.8)
- moved D1 0.50 mm to (91.0, 66.7), turned to 90 degrees
Routing:
- net +5V: track 0.00 -> 28.0 mm, vias 0 -> 1
- net /TPIDATA: track 0.00 -> 27.8 mm, vias 0 -> 2
- net GND: track 0.00 -> 23.4 mm, vias 0 -> 22
- net /TPICLK: track 0.00 -> 16.5 mm, vias 0 -> 2
- net +12V: track 4.49 -> 17.3 mm
- net /LED_DATA: track 0.00 -> 7.06 mm
- net /~{RESET}: track 0.00 -> 7.03 mm, vias 0 -> 1
- net /FAN_PWM_OD: track 0.00 -> 3.63 mm
- added copper zone on F.Cu, net GND
Other:
- board size 17.4 x 26.9 mm -> 17.4 x 27 mm
