File: pwm-fan-control.kicad_sch (KiCad schematic)
At the start: 13 parts, among them J1 12V_IN, J2 FAN_OUT, J3 Conn_ESP_PROG_1.27mm_TagConne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, J4 ADJ_IN, Q1 NMOS (100V 1.5A 2Vth), U1 NCP1117-5.0_SOT223, U2 ATtiny10-TS

Commit message: Plot PDF schematic
Other:
- company: (none) -> GIE Design
- title: (none) -> PWM Fan Controller
Changed lines of the file:
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@@
 (kicad_sch (version 20210621) (generator eeschema)
   (paper "A4")
+  (title_block
+    (title "PWM Fan Controller")
+    (date "2021-10-19")
+    (rev "1")
+    (company "GIE Design")
+  )
   (junction (at 40.64 76.2) (diameter 0) (color 0 0 0 0))
   (junction (at 45.72 73.66) (diameter 0) (color 0 0 0 0))
